File: bp-sideview.sch (KiCad schematic (older format))
At the start: 7 parts

Commit message: time to lay this sucker out
Parts:
- added D10, D11, D12, D13, D14, D15, D16, D17, D18, D19, D20, D4, D5, D6, D7, D8, D9: LED, LED_SMD:LED_1206_3216Metric, symbol Device:LED
- added R10, R11, R12, R13, R14, R15, R16, R17, R18, R19, R20, R4, R5, R6, R7, R8, R9: 1K, Resistor_SMD:R_0603_1608Metric, symbol Device:R
- BT1: footprint (none) -> Battery:BatteryHolder_MPD_BC2003_1x2032
Connections:
- net GND: now also D10.1 (K), D11.1 (K), D12.1 (K), D13.1 (K), D14.1 (K), D15.1 (K), D16.1 (K), D17.1 (K), D18.1 (K), D19.1 (K), D20.1 (K), D4.1 (K), D5.1 (K), D6.1 (K), D7.1 (K), D8.1 (K), D9.1 (K), R10.2, R11.2, R12.2, R13.2, R14.2, R15.2, R16.2, R17.2, R18.2, R19.2, R20.2, R4.2, R5.2, R6.2, R7.2, R8.2, R9.2
- new net: D4.2 (A), R4.1
- new net: D5.2 (A), R5.1
- new net: D6.2 (A), R6.1
- new net: D7.2 (A), R7.1
- new net: D8.2 (A), R8.1
- new net: D9.2 (A), R9.1
- new net: D10.2 (A), R10.1
- new net: D11.2 (A), R11.1
- new net: D12.2 (A), R12.1
- new net: D13.2 (A), R13.1
- new net: D14.2 (A), R14.1
- new net: D15.2 (A), R15.1
- new net: D16.2 (A), R16.1
- new net: D17.2 (A), R17.1
- new net: D20.2 (A), R20.1
- new net: D19.2 (A), R19.1
- new net: D18.2 (A), R18.1
Other:
- moved on the sheet: D1, D2, D3, R1, R2, R3
